File: D1MPOWER.brd (EAGLE design)
At the start: 25.4 x 33 mm, 11 parts, among them IC3 MC33269DT-5.0, J5 DC_2_1MM

Commit message: Optimised part designators
Parts:
- renumbered C10 to C2, C5 to C3, IC3 to IC1, J5 to J2, JP1 to J1
Changed lines of the file:
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@@
 <attribute name="VALUE" x="20.955" y="27.94" size="1.27" layer="27" rot="R270"/>
 </element>
-<element name="J5" library="freetronics" package="POWER_JACK_PTH" value="DC_2_1MM" x="7.62" y="-1.27"/>
-<element name="IC3" library="linear" package="DPACK" value="MC33269DT-5.0" x="16.51" y="19.05" rot="R180"/>
+<element name="J2" library="freetronics" package="POWER_JACK_PTH" value="DC_2_1MM" x="7.62" y="-1.27"/>
+<element name="IC1" library="linear" package="DPACK" value="MC33269DT-5.0" x="16.51" y="19.05" rot="R180"/>
 <element name="C1" library="rcl" package="PANASONIC_D" value="47uF 25V" x="7.62" y="29.21"/>
-<element name="C5" library="rcl" package="PANASONIC_D" value="47uF 25V" x="17.78" y="29.21"/>
+<element name="C3" library="rcl" package="PANASONIC_D" value="47uF 25V" x="17.78" y="29.21"/>
 <element name="D1" library="freetronics" package="SMB-DIODE" value="1N4004 SMB" x="7.62" y="20.32" rot="R270"/>
-<element name="C10" library="freetronics" package="0603" value="100nF 0603" x="20.32" y="11.43"/>
+<element name="C2" library="freetronics" package="0603" value="100nF 0603" x="20.32" y="11.43"/>
 <element name="LED1" library="freetronics-jon" package="LED-0603" value="BLUE" x="23.622" y="4.826" rot="R90"/>
 <element name="R1" library="freetronics-jon" package="0603" value="2K2" x="16.51" y="11.43"/>
-<element name="JP1" library="freetronics-jon" package="SCREWTERMINAL-3.5MM-2" value="" x="20.32" y="6.35" rot="R180"/>
+<element name="J1" library="freetronics-jon" package="SCREWTERMINAL-3.5MM-2" value="" x="20.32" y="6.35" rot="R180"/>
 </elements>
 <signals>
@@
 <contactref element="H2" pad="7"/>
 <contactref element="C1" pad="-"/>
-<contactref element="J5" pad="GNDBREAK"/>
-<contactref element="J5" pad="GND"/>
-<contactref element="IC3" pad="1"/>
-<contactref element="C10" pad="2"/>
-<contactref element="C5" pad="-"/>
+<contactref element="J2" pad="GNDBREAK"/>
+<contactref element="J2" pad="GND"/>
+<contactref element="IC1" pad="1"/>
+<contactref element="C2" pad="2"/>
+<contactref element="C3" pad="-"/>
 <contactref element="LED1" pad="C"/>
-<contactref element="JP1" pad="1"/>
+<contactref element="J1" pad="1"/>
 </signal>
 <signal name="D1">
@@
 <signal name="5V">
 <contactref element="H2" pad="8"/>
-<contactref element="C5" pad="+"/>
-<contactref element="IC3" pad="2"/>
-<contactref element="C10" pad="1"/>
+<contactref element="C3" pad="+"/>
+<contactref element="IC1" pad="2"/>
+<contactref element="C2" pad="1"/>
 <contactref element="R1" pad="2"/>
 <wire x1="20.18" y1="29.21" x2="20.18" y2="27.8" width="0.8128" layer="1"/>
@@
 <signal name="VIN">
 <contactref element="D1" pad="C"/>
-<contactref element="IC3" pad="3"/>
+<contactref element="IC1" pad="3"/>
 <contactref element="C1" pad="+"/>
 <wire x1="7.62" y1="22.52" x2="8.95" y2="23.85" width="0.8128" layer="1"/>
@@
 </signal>
 <signal name="N$8">
-<contactref element="J5" pad="PWR"/>
+<contactref element="J2" pad="PWR"/>
 <contactref element="D1" pad="A"/>
-<contactref element="JP1" pad="2"/>
+<contactref element="J1" pad="2"/>
 <wire x1="16.82" y1="6.35" x2="11.176" y2="6.35" width="0.8128" layer="1"/>
 <wire x1="11.176" y1="6.35" x2="8.89" y2="9.398" width="0.8128" layer="1"/>
